Commit message: refactor Gazebo-Rviz-TF tutorials

File: source/_static/scripts/simplexacro.xacro (robot description, xacro)
@@ -1,5 +1,5 @@
 <?xml version="1.0"?>
-<robot name="multipleshapes">
-  <link name="base_link">
+<robot name="myrobot">
+  <link name="link1">
     <visual>
       <geometry>
@@ -8,5 +8,5 @@
     </visual>
   </link>
-  <link name="right_leg">
+  <link name="link2">
     <visual>
       <geometry>
@@ -15,7 +15,7 @@
     </visual>
   </link>
-  <joint name="base_to_right_leg" type="fixed">
-    <parent link="base_link"/>
-    <child link="right_leg"/>
+  <joint name="link1_to_link2" type="fixed">
+    <parent link="link1"/>
+    <child link="link2"/>
   </joint>
 </robot>
